File: GameBoy-Arduino.kicad_pcb (KiCad board)
At the start: 2 copper layers, 106.3 x 39.5 mm, 26 parts, among them SW1 SW_Push_Open, SW2 SW_Push_Open, SW3 SW_Push_Open, SW4 SW_Push_Open, SW5 SW_Push_Open, SW6 SW_Push_Open, SW7 SW_SPDT, U1 TP4056, U2 MT3608, U4 Arduino Pro Micro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

Commit message: updated silkscreen
Parts:
- removed the G*** at (99.2, 83.6)
- removed kibuzzard-653E884F: G***, kibuzzard-653E884F
Other:
- board text added: "**REDACTED PROTOTYPE: LED MATRIX GAME**"
- board text removed: "**NINTENDO PROTOTYPE: LED MATRIX GAME**"
- board text removed: "Actually it's not Nintendo pls don't sue"
